File: sch/power_mng.kicad_sch (KiCad schematic)
At the start: 27 parts, among them J1 USB_C_Receptacle_USB2.0_16P, U2 TPS63061, U3 USBLC6-2P6, U5 TLV75801PDRV, U6 TLV75533PDRV

Commit message: routes
Parts:
- added H1, H2, H3, H4: MountingHole, MountingHole:MountingHole_3.2mm_M3, symbol Mechanical:MountingHole
- added J3: Batt-Con, Connector_AMASS:AMASS_XT30PW-M_1x02_P2.50mm_Horizontal, symbol Connector_Generic:Conn_01x02
Connections:
- net +BATT renamed +8V4
- net +8V4: now also J3.1 (Pin_1)
- net -BATT renamed GND
- net GND: now also J3.2 (Pin_2)
