File: sch/power_mng.kicad_sch (KiCad schematic)
At the start: 32 parts, among them J1 USB_C_Receptacle_USB2.0_16P, J3 Batt-Con, U2 TPS63061, U3 USBLC6-2P6, U5 TLV75801PDRV, U6 TLV75533PDRV

Commit message: MSD card, mag, imu
this thang gonna cost so much money
Parts:
- removed H1, H2, H3, H4: MountingHole, MountingHole:MountingHole_3.2mm_M3, symbol Mechanical:MountingHole

Commit message: gah
Parts:
- removed D1, D2: PMEG2010ET, Package_TO_SOT_SMD:SOT-23, symbol Diode:PMEG2010ET
- removed R10: 111kR, Resistor_SMD:R_0402_1005Metric, symbol Device:R_Small_US
- removed R9: 1MR, Resistor_SMD:R_0402_1005Metric, symbol Device:R_Small_US
- added D5, D6: PMEG2010ER, Diode_SMD:Nexperia_CFP3_SOD-123W, symbol Diode:PMEG2010ER
- C3, C4, C5, C6: footprint Capacitor_SMD:C_0201_0603Metric -> Capacitor_SMD:C_01005_0402Metric
- F1: footprint Fuse:Fuse_0402_1005Metric -> Fuse:Fuse_0603_1608Metric
Connections:
- net +8V4: now also D5.2 (A)
- net V_OUT: now also C10.1, U2.8 (FB), D6.1 (K)
- net at F1.2, U3.5 (VBUS): now also D6.2 (A)
- net at C8.1, U2.2 (VIN), U2.3 (EN): now also D5.1 (K)
Other:
- moved on the sheet: C10, C11, C12, C13, C7, C8, C9, L1, R11, U2

Commit message: reroute
doooom
Connections:
- net +DVDD: now also C6.1; no longer C6.2
- net GND: now also C6.2; no longer C6.1
Changed lines of the file:
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@@
 		(lib_id "Device:C_Small")
 		(at 99.06 128.27 0)
-		(mirror x)
 		(unit 1)
 		(body_style 1)
@@
 		(dnp no)
 		(property "Reference" "C6"
-			(at 101.6 129.5338 0)
+			(at 101.6 127.0062 0)
 			(show_name no)
 			(do_not_autoplace no)
@@
 		)
 		(property "Value" "1uF"
-			(at 101.6 126.9938 0)
+			(at 101.6 129.5462 0)
 			(show_name no)
 			(do_not_autoplace no)

Commit message: footprints
Parts:
- C11, C12, C13: footprint Capacitor_SMD:C_0402_1005Metric -> Capacitor_SMD:C_0603_1608Metric
- C3, C4, C5, C6: footprint Capacitor_SMD:C_01005_0402Metric -> Capacitor_SMD:C_0402_1005Metric
- L1: footprint Inductor_SMD:L_0402_1005Metric -> Inductor_SMD:L_Coilcraft_XxL4020
- R11: value 1MR -> 100kR
Changed lines of the file:
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@@
 			)
 		)
-		(property "Footprint" "Capacitor_SMD:C_0402_1005Metric"
+		(property "Footprint" "Capacitor_SMD:C_0603_1608Metric"
 			(at 229.87 72.39 0)
 			(hide yes)
@@
 			)
 		)
-		(property "Footprint" "Capacitor_SMD:C_0402_1005Metric"
+		(property "Footprint" "Capacitor_SMD:C_0603_1608Metric"
 			(at 229.87 67.31 0)
 			(hide yes)
@@
 			)
 		)
-		(property "Footprint" "Capacitor_SMD:C_0402_1005Metric"
+		(property "Footprint" "Capacitor_SMD:C_0603_1608Metric"
 			(at 229.87 77.47 0)
 			(hide yes)
@@
 			)
 		)
-		(property "Footprint" "Capacitor_SMD:C_01005_0402Metric"
+		(property "Footprint" "Capacitor_SMD:C_0402_1005Metric"
 			(at 99.06 128.27 0)
 			(hide yes)
@@
 			)
 		)
-		(property "Footprint" "Capacitor_SMD:C_01005_0402Metric"
+		(property "Footprint" "Capacitor_SMD:C_0402_1005Metric"
 			(at 170.18 129.54 0)
 			(hide yes)
@@
 			)
 		)
-		(property "Footprint" "Capacitor_SMD:C_01005_0402Metric"
+		(property "Footprint" "Capacitor_SMD:C_0402_1005Metric"
 			(at 144.78 129.54 0)
 			(hide yes)
@@
 			)
 		)
-		(property "Footprint" "Capacitor_SMD:C_01005_0402Metric"
+		(property "Footprint" "Capacitor_SMD:C_0402_1005Metric"
 			(at 72.39 128.27 0)
 			(hide yes)
@@
 			)
 		)
-		(property "Value" "1MR"
+		(property "Value" "100kR"
 			(at 218.44 73.6599 0)
 			(show_name no)
@@
 			)
 		)
-		(property "Footprint" "Inductor_SMD:L_0402_1005Metric"
+		(property "Footprint" "Inductor_SMD:L_Coilcraft_XxL4020"
 			(at 157.48 80.01 0)
 			(hide yes)

Commit message: v1.1e for real
ordered!
Redid high power side.
Added breakouts for power and the motor driver.
Parts:
- added J10: Power_Pins, Connector_PinHeader_2.54mm:PinHeader_2x03_P2.54mm_Vertical, symbol Connector_Generic:Conn_02x03_Odd_Even
Connections:
- net +3V3: now also J10.3 (Pin_3)
- net +DVDD: now also J10.5 (Pin_5)
- net GND: now also J10.2 (Pin_2), J10.4 (Pin_4), J10.6 (Pin_6)
- net V_OUT: now also J10.1 (Pin_1)
