File: rp2354b-fast.kicad_pcb (KiCad board)
At the start: 2 copper layers, 49 parts, among them J1 USB_C_Receptacle_USB2.0_16P, J2 Conn_ARM_SWD_TagConnect_TC203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, SW1 SW_Push, SW2 SW_Push, U1 RP2354B, U2 TPS63061, U3 USBLC6-2P6, U5 TLV75801PDRV, U6 TLV75533PDRV, Y1 12MHz

Commit message: routes
Parts:
- added C21: 100nF, Capacitor_SMD:C_0402_1005Metric, F.Cu at (153.2, 99.5)
- added C22: 100nF, Capacitor_SMD:C_0402_1005Metric, F.Cu at (152.2, 99.5)
- added C26: 100nF, Capacitor_SMD:C_0402_1005Metric, F.Cu at (157.3, 99.5)
- added C27: 100nF, Capacitor_SMD:C_0402_1005Metric, F.Cu at (160.8, 111.0)
- added H1: MountingHole, MountingHole:MountingHole_3.2mm_M3, F.Cu at (159.7, 139.2)
- added H2: MountingHole, MountingHole:MountingHole_3.2mm_M3, F.Cu at (159.7, 94.8)
- added H3: MountingHole, MountingHole:MountingHole_3.2mm_M3, F.Cu at (115.3, 94.8)
- added H4: MountingHole, MountingHole:MountingHole_3.2mm_M3, F.Cu at (115.3, 139.2)
- added J3: Batt-Con, Connector_AMASS:AMASS_XT30PW-M_1x02_P2.50mm_Horizontal, F.Cu at (115.4, 114.6)
- moved R3 127.8 mm to (163.8, 108.4), turned to -90 degrees
- moved SW2 124.2 mm to (167.2, 109.9), turned to 180 degrees
- moved C2 123.6 mm to (154.9, 117.9), turned to 180 degrees
- moved C1 123.1 mm to (152.9, 117.9)
- moved J2 121.8 mm to (165.9, 114.6), turned to 180 degrees
- moved C20 118.9 mm to (160.8, 107.0)
- moved D3 118.7 mm to (165.7, 118.7)
- moved R1 118.1 mm to (155.3, 99.5), turned to 90 degrees
- moved C14 117.2 mm to (150.6, 114.8), turned to -90 degrees
- moved R2 116.2 mm to (154.2, 99.5), turned to 90 degrees
- moved C25 116.1 mm to (156.3, 114.8), turned to -90 degrees
- moved C15 115.2 mm to (149.5, 114.8), turned to -90 degrees
- moved Y1 110.7 mm to (153.7, 115.7)
- moved C23 110.4 mm to (156.3, 99.5), turned to 90 degrees
- moved R4 108.8 mm to (147.5, 100.4), turned to 90 degrees
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Connections:
- C10 pad 2: -BATT -> GND
- C13 pad 2: -BATT -> GND
- C14 pad 2: -BATT -> GND
- C15 pad 2: -BATT -> GND
- C16 pad 2: -BATT -> GND
- C17 pad 2: -BATT -> GND
- C18 pad 2: -BATT -> GND
- C19 pad 2: -BATT -> GND
- C20 pad 2: -BATT -> GND
- C23 pad 2: -BATT -> GND
- C24 pad 2: -BATT -> GND
- C25 pad 2: -BATT -> GND
- C3 pad 2: -BATT -> GND
- C4 pad 2: -BATT -> GND
- C5 pad 2: -BATT -> GND
- C6 pad 1: -BATT -> GND
- C7 pad 2: -BATT -> GND
- C9 pad 2: -BATT -> GND
- D2 pad 1: +BATT -> +8V4
- D3 pad 2: -BATT -> GND
- J1 pad A1: -BATT -> GND
- J1 pad A12: -BATT -> GND
- J1 pad A6: /power_mng/D+ -> /D+
- J1 pad A7: /power_mng/D- -> /D-
- J1 pad B1: -BATT -> GND
- J1 pad B12: -BATT -> GND
- J1 pad B6: /power_mng/D+ -> /D+
- J1 pad B7: /power_mng/D- -> /D-
- J1 pad SH: -BATT -> GND
- J2 pad 5: -BATT -> GND
- R10 pad 1: -BATT -> GND
- R5 pad 1: -BATT -> GND
- R6 pad 1: -BATT -> GND
- R8 pad 1: -BATT -> GND
- SW1 pad 1: -BATT -> GND
- SW2 pad 1: -BATT -> GND
- U1 pad 10: -BATT -> +DVDD
- U1 pad 15: -BATT -> +3V3
- U1 pad 24: -BATT -> +3V3
- U1 pad 29: -BATT -> +3V3
- U1 pad 32: -BATT -> +DVDD
- U1 pad 41: -BATT -> +3V3
- U1 pad 5: -BATT -> +3V3
- U1 pad 50: -BATT -> +3V3
- U1 pad 51: -BATT -> +DVDD
- U1 pad 59: -BATT -> +3V3
- U1 pad 60: -BATT -> +3V3
- U1 pad 61: -BATT -> +3V3
- U1 pad 62: -BATT -> GND
- U1 pad 64: -BATT -> GND
- U1 pad 65: -BATT -> +DVDD
- U1 pad 68: -BATT -> +3V3
- U1 pad 69: -BATT -> +3V3
- U1 pad 76: -BATT -> +3V3
- U1 pad 81: -BATT -> GND
- U2 pad 11: -BATT -> GND
- U2 pad 4: -BATT -> GND
- U2 pad 7: -BATT -> GND
- U3 pad 1: /power_mng/D+ -> /D+
- U3 pad 2: -BATT -> GND
- U3 pad 3: /power_mng/D- -> /D-
- U3 pad 4: /power_mng/D- -> /D-
- U3 pad 6: /power_mng/D+ -> /D+
- U5 pad 3: -BATT -> GND
- U5 pad 7: -BATT -> GND
- U6 pad 3: -BATT -> GND
- U6 pad 7: -BATT -> GND
- Y1 pad 2: -BATT -> GND
- Y1 pad 4: -BATT -> GND
Routing:
- net +3V3: track 0.00 -> 116.8 mm, vias 0 -> 4
- net GND: track 0.00 -> 80.9 mm, vias 0 -> 37
- net +DVDD: track 0.00 -> 55.2 mm, vias 0 -> 4
- net Net-(D1-K): track 0.00 -> 41.3 mm, vias 0 -> 2
- net /D+: track 0.00 -> 28.7 mm
- net V_OUT: track 0.00 -> 26.9 mm, vias 0 -> 2
- net /D-: track 0.00 -> 26.8 mm
- net /~{RESET}: track 0.00 -> 26.7 mm, vias 0 -> 2
- net Net-(J2-SWCLK): track 0.00 -> 15.2 mm
- net Net-(U1-~{QSPI_SS}): track 0.00 -> 14.9 mm, vias 0 -> 2
- net Net-(J2-SWDIO): track 0.00 -> 14.4 mm
- net Net-(F1-Pad1): track 0.00 -> 10.2 mm
- net Net-(D1-A): track 0.00 -> 9.55 mm, vias 0 -> 3
- net Net-(U1-XOUT): track 0.00 -> 6.91 mm
- net Net-(U1-XIN): track 0.00 -> 6.81 mm
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Other:
- board outline added: 70 x 70 mm
- copper layers 2 -> 4

Commit message: footprint
Routing:
- net GND: track 80.9 -> 95.5 mm, vias 37 -> 42
- net +3V3: track 116.8 -> 120.9 mm, vias 4 -> 6
- net Net-(C11-Pad2): track 0.00 -> 1.01 mm
- net Net-(C12-Pad2): track 0.00 -> 1.00 mm
- added copper zone on In1.Cu, net GND

Commit message: routes and bmp581
Parts:
- added C28: 100nF, Capacitor_SMD:C_0402_1005Metric, F.Cu at (143.0, 111.8)
- added C29: 100nF, Capacitor_SMD:C_0402_1005Metric, F.Cu at (144.9, 113.5)
- added U4: BMP581, footprints:QFN10_BMP581_BOS-L, F.Cu at (145.2, 111.3)
- moved C24 15.0 mm to (160.8, 107.0), turned to 0 degrees
- moved C20 14.2 mm to (146.6, 107.0), turned to 180 degrees
- moved SW1 4.05 mm to (142.7, 100.5)
- moved C19 2.19 mm to (144.1, 109.0)
- moved C18 1.90 mm to (149.3, 99.5)
- moved C22 1.30 mm to (150.9, 99.5)
- moved R4 0.92 mm to (147.7, 99.5), turned to -90 degrees
- moved C16 0.80 mm to (146.6, 105.0)
- moved C17 0.80 mm to (146.6, 109.0)
- moved C15 0.70 mm to (148.8, 114.8)
- moved C21 0.70 mm to (152.5, 99.5)
Connections:
- U1 pad 16: unconnected-(U1-GPIO16-Pad16) -> GPIO16_SPI0_RX
- U1 pad 17: unconnected-(U1-GPIO17-Pad17) -> GPIO17_SPI0_CSN
- U1 pad 18: unconnected-(U1-GPIO18-Pad18) -> GPIO18_SPI0_SCK
- U1 pad 19: unconnected-(U1-GPIO19-Pad19) -> GPIO19_SPI0_TX
- U1 pad 20: unconnected-(U1-GPIO20-Pad20) -> GPIO20_SPI0_RX
- U1 pad 21: unconnected-(U1-GPIO21-Pad21) -> GPIO21_SPI0_CSN
- U1 pad 22: unconnected-(U1-GPIO22-Pad22) -> GPIO22SPI0_SCK
- U1 pad 23: unconnected-(U1-GPIO23-Pad23) -> GPIO23_SPI0_TX
Routing:
- net +3V3: track 120.9 -> 65.9 mm, vias 6 -> 19
- net +DVDD: track 55.2 -> 78.0 mm
- net GND: track 95.5 -> 87.0 mm, vias 42 -> 51
- net GPIO18_SPI0_SCK: track 0.00 -> 7.38 mm, vias 0 -> 2
- net GPIO17_SPI0_CSN: track 0.00 -> 3.26 mm, vias 0 -> 2
- net GPIO16_SPI0_RX: track 0.00 -> 3.25 mm
- net GPIO19_SPI0_TX: track 0.00 -> 2.54 mm
- net /D-: track 26.8 -> 28.2 mm
- net Net-(U4-V_DD): track 0.00 -> 0.99 mm
- net /D+: track 28.7 -> 29.3 mm
- net Net-(U1-~{QSPI_SS}): track 14.9 -> 15.5 mm
- added copper zone on In2.Cu, net +3V3

Commit message: hv16v
Parts:
- added J4: XT60 Male, Connector_AMASS:AMASS_XT60IPW-M_1x03_P7.20mm_Horizontal, F.Cu at (141.1, 135.6)
- added U7: DRV8461SPWP, Package_SO:Texas_PWP0020A, F.Cu at (153.9, 130.3)
- added U8: LSM9DS1, Package_LGA:LGA-24L_3x3.5mm_P0.43mm, F.Cu at (137.5, 117.0)
- J2: value Conn_ARM_SWD_TagConnect_TC2030-NL -> TC2030-Tag
- moved D3 0.80 mm to (166.5, 118.7)
Connections:
- net /power_mng/FB renamed /power_mng_3v3/FB
- net /power_mng/PG renamed /power_mng_3v3/PG
- D3 pad 3: unconnected-(D3-DIN-Pad3) -> GPIO33_LED
- R3 pad 2: /~{RESET} -> Net-(R3-Pad2)
- SW2 pad 2: /~{RESET} -> Net-(R3-Pad2)
- U1 pad 42: unconnected-(U1-GPIO33-Pad42) -> GPIO33_LED
Routing:
- net GND: track 87.0 -> 62.3 mm, vias 51 -> 50
- net +DVDD: track 78.0 -> 53.7 mm
- net GPIO33_LED: track 0.00 -> 14.6 mm, vias 0 -> 2
- net Net-(D1-K): track 41.3 -> 46.8 mm
- net /~{RESET}: track 26.7 -> 24.1 mm, vias 2 -> 0
- net +3V3: track 65.9 -> 68.1 mm
- net Net-(U1-~{QSPI_SS}): track 15.5 -> 14.3 mm, vias 2 -> 0
- net Net-(F1-Pad1): track 10.2 -> 9.47 mm
- net V_OUT: track 26.9 -> 27.4 mm

Commit message: imu sym
Parts:
- removed J4: XT60 Male, Connector_AMASS:AMASS_XT60IPW-M_1x03_P7.20mm_Horizontal
- removed U8: LSM9DS1, Package_LGA:LGA-24L_3x3.5mm_P0.43mm
- added C30: 220uF, Capacitor_SMD:CP_Elec_8x10, F.Cu at (129.7, 121.7)
- added C31: 100nF, Capacitor_SMD:C_0402_1005Metric, F.Cu at (111.9, 134.1)
- added C32: 1uF, Capacitor_SMD:C_0402_1005Metric, F.Cu at (111.3, 132.6)
- added C33: 100uF, Capacitor_SMD:C_1206_3216Metric, F.Cu at (122.5, 126.2)
- added C34: 1uF, Capacitor_SMD:C_0402_1005Metric, F.Cu at (110.8, 126.4)
- added C35: 10nF, Capacitor_SMD:C_1206_3216Metric, F.Cu at (125.4, 129.5)
- added C36: 10nF, Capacitor_SMD:C_1206_3216Metric, F.Cu at (122.5, 133.2)
- added C37: 1uF, Capacitor_SMD:C_1206_3216Metric, F.Cu at (120.0, 137.3)
- added C38: 1uF, Capacitor_SMD:C_0402_1005Metric, F.Cu at (111.4, 128.1)
- added D4: SMCJ18CA, PCM_JLCPCB:D_SMC, F.Cu at (137.6, 129.6)
- added J5: STPR_OUT, Connector_JST:JST_XA_B04B-XASK-1_1x04_P2.50mm_Vertical, F.Cu at (125.5, 145.2)
- added J6: Conn_01x03_Socket, Connector_AMASS:AMASS_XT60IPW-M_1x03_P7.20mm_Horizontal, F.Cu at (141.1, 135.6)
- added R14: 10kR, Resistor_SMD:R_0402_1005Metric, F.Cu at (111.9, 126.4)
- J3: moved to B.Cu
- U4: footprint footprints:QFN10_BMP581_BOS-L -> BMP581:QFN10_BMP581_BOS
- U7: footprint Package_SO:Texas_PWP0020A -> Package_SO:HTSSOP-28-1EP_4.4x9.7mm_P0.65mm_EP2.85x5.4mm_ThermalVias
- moved U7 37.6 mm to (116.3, 129.7), turned to 180 degrees
- moved D2 11.7 mm to (116.7, 104.4), turned to 90 degrees
- moved J3 7.30 mm to (120.2, 109.2), turned to -90 degrees
Connections:
- net GPIO33_LED renamed /GPIO33_LED
- net Net-(U7-AOUT1-Pad4) renamed /HV_16v8/AOUT1
- net Net-(U7-AOUT2-Pad6) renamed /HV_16v8/AOUT2
- net Net-(U7-BOUT1-Pad10) renamed /HV_16v8/BOUT1
- net Net-(U7-BOUT2-Pad8) renamed /HV_16v8/BOUT2
- net Net-(U7-VM-Pad13) renamed +16V8
- U1 pad 20: GPIO20_SPI0_RX -> /GPIO20_SPI0_RX
- U1 pad 21: GPIO21_SPI0_CSN -> /GPIO21_SPIO_CSN
- U1 pad 22: GPIO22SPI0_SCK -> /GPIO22_SPIO_SCK
- U1 pad 23: GPIO23_SPI0_TX -> /GPIO23_SPIO_TX
- U1 pad 25: unconnected-(U1-GPIO24-Pad25) -> /STPER_ENABLE
- U1 pad 26: unconnected-(U1-GPIO25-Pad26) -> /STPER_DIR
- U1 pad 27: unconnected-(U1-GPIO26-Pad27) -> /STPER_STEP
- U7 pad 1: unconnected-(U7-VCP-Pad1) -> Net-(U7-VCP)
- U7 pad 12: Net-(U7-GND-Pad12) -> GND
- U7 pad 14: Net-(U7-GND-Pad12) -> GND
- U7 pad 15: unconnected-(U7-DVDD-Pad15) -> /HV_16v8/DVDD
- U7 pad 16: unconnected-(U7-~{FAULT}-Pad16) -> Net-(U7-~{FAULT})
- U7 pad 17: unconnected-(U7-VREF-Pad17) -> +3V3
- U7 pad 18: unconnected-(U7-~{SCS}-Pad18) -> /GPIO21_SPIO_CSN
- U7 pad 19: unconnected-(U7-VCC-Pad19) -> +3V3
- U7 pad 20: unconnected-(U7-SDO-Pad20) -> /GPIO20_SPI0_RX
- U7 pad 21: unconnected-(U7-SDI-Pad21) -> /GPIO23_SPIO_TX
- U7 pad 3: Net-(U7-GND-Pad12) -> GND
Routing:
- net /STPER_STEP: track 0.00 -> 57.0 mm, vias 0 -> 2
- net /STPER_DIR: track 0.00 -> 55.8 mm, vias 0 -> 4
- net /STPER_ENABLE: track 0.00 -> 54.1 mm, vias 0 -> 2
- net /GPIO22_SPIO_SCK: track 0.00 -> 49.8 mm, vias 0 -> 2
- net /GPIO23_SPIO_TX: track 0.00 -> 49.2 mm, vias 0 -> 4
- net /GPIO21_SPIO_CSN: track 0.00 -> 45.5 mm
- net /GPIO20_SPI0_RX: track 0.00 -> 43.1 mm, vias 0 -> 2
- net +3V3: track 68.1 -> 106.9 mm, vias 19 -> 22
- net /HV_16v8/BOUT2: track 0.00 -> 19.8 mm
- net /HV_16v8/BOUT1: track 0.00 -> 17.6 mm, vias 0 -> 1
- net /HV_16v8/AOUT1: track 0.00 -> 16.8 mm, vias 0 -> 1
- net /HV_16v8/AOUT2: track 0.00 -> 15.9 mm, vias 0 -> 1
- net GND: track 62.3 -> 74.0 mm, vias 50 -> 65
- net /~{RESET}: track 24.1 -> 12.4 mm
- net Net-(D1-K): track 46.8 -> 35.6 mm
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- added copper zone on In2.Cu, net +16V8
