File: rp2354b-fast.kicad_pcb (KiCad board)
At the start: 4 copper layers, 70 x 70 mm, 75 parts, among them J1 USB_C_Receptacle_USB2.0_16P, J2 TC2030-Tag, J3 Batt-Con, J5 STPR_OUT, J6 Conn_01x03_Socket, SW1 SW_Push, SW2 SW_Push, U1 RP2354B, U2 TPS63061, U3 USBLC6-2P6, U4 BMP581, U5 TLV75801PDRV, U6 TLV75533PDRV, U7 DRV8461SPWP, Y1 12MHz

Commit message: MSD card, mag, imu
this thang gonna cost so much money
Parts:
- added C39: 100nF, Capacitor_SMD:C_0402_1005Metric, F.Cu at (136.3, 119.5)
- added C40: 100nF, Capacitor_SMD:C_0402_1005Metric, F.Cu at (140.2, 117.9)
- added C41: 1uF, Capacitor_SMD:C_0402_1005Metric, F.Cu at (165.3, 100.2)
- added C42: 10uF, Capacitor_SMD:C_0402_1005Metric, F.Cu at (167.8, 102.7)
- added C43: 100nF, Capacitor_SMD:C_0402_1005Metric, F.Cu at (162.8, 102.8)
- added C44: 10uF, Capacitor_SMD:C_0402_1005Metric, B.Cu at (155.8, 122.5)
- added C45: 100nF, Capacitor_SMD:C_0402_1005Metric, B.Cu at (155.6, 127.7)
- added J4: MSD-10-C, MSD-10-C:MSD-10-C, F.Cu at (155.6, 127.6)
- added R12: 10kR, Resistor_SMD:R_0402_1005Metric, B.Cu at (152.4, 122.5)
- added R13: 10kR, Resistor_SMD:R_0402_1005Metric, B.Cu at (160.1, 127.7)
- added R15: 10kR, Resistor_SMD:R_0402_1005Metric, B.Cu at (159.0, 127.7)
- added R16: 10kR, Resistor_SMD:R_0402_1005Metric, B.Cu at (156.8, 127.7)
- added R17: 10kR, Resistor_SMD:R_0402_1005Metric, B.Cu at (154.6, 127.7)
- added R18: 10kR, Resistor_SMD:R_0402_1005Metric, B.Cu at (153.5, 127.7)
- added U8: ISM6HG256X, Package_LGA:LGA-14_3x2.5mm_P0.5mm_LayoutBorder3x4y, F.Cu at (137.5, 117.0)
- added U9: MMC5983MA, Package_LGA:LGA-16_3x3mm_P0.5mm, F.Cu at (165.1, 102.5)
- J3: moved to F.Cu
- moved H1 62.8 mm to (115.3, 94.8)
- moved H3 62.8 mm to (159.7, 139.2)
- moved D2 5.71 mm to (122.4, 104.8)
- moved J3 3.31 mm to (118.3, 106.5), turned to 90 degrees
- moved C24 1.08 mm to (159.7, 107.0)
Connections:
- net GPIO16_SPI0_RX renamed /GPIO16_SPI0_RX
- net GPIO17_SPI0_CSN renamed /GPIO17_SPI0_CSN
- net GPIO18_SPI0_SCK renamed /GPIO18_SPI0_SCK
- net GPIO19_SPI0_TX renamed /GPIO19_SPI0_TX
- R3 pad 2: Net-(R3-Pad2) -> /~{RESET}
- SW2 pad 2: Net-(R3-Pad2) -> /~{RESET}
- U1 pad 14: unconnected-(U1-GPIO15-Pad14) -> /GPIO14_CSN_IMU
- U1 pad 36: unconnected-(U1-GPIO28-Pad36) -> /GPIO28_SD_CS
- U1 pad 45: unconnected-(U1-GPIO36-Pad45) -> /GPIO36_RX
- U1 pad 46: unconnected-(U1-GPIO37-Pad46) -> /GPIO37_CSN
- U1 pad 47: unconnected-(U1-GPIO38-Pad47) -> /GPIO38_SCK
- U1 pad 48: unconnected-(U1-GPIO39-Pad48) -> /GPIO39_TX
Routing:
- net /GPIO16_SPI0_RX: track 3.25 -> 50.8 mm, vias 0 -> 4
- net /GPIO19_SPI0_TX: track 2.54 -> 41.6 mm, vias 0 -> 4
- net /GPIO18_SPI0_SCK: track 7.51 -> 42.1 mm, vias 2 -> 5
- net +3V3: track 106.9 -> 125.2 mm, vias 22 -> 34
- net /GPIO14_CSN_IMU: track 0.00 -> 17.5 mm, vias 0 -> 2
- net /GPIO28_SD_CS: track 0.00 -> 15.8 mm, vias 0 -> 3
- net GND: track 74.0 -> 88.3 mm, vias 65 -> 81
- net /GPIO39_TX: track 0.00 -> 13.2 mm
- net /GPIO38_SCK: track 0.00 -> 12.7 mm
- net /~{RESET}: track 12.4 -> 22.3 mm, vias 0 -> 3
- net /GPIO36_RX: track 0.00 -> 9.83 mm
- net /GPIO37_CSN: track 0.00 -> 9.62 mm
- net Net-(D1-K): track 35.6 -> 41.4 mm
- net Net-(R3-Pad2): track 5.51 -> 0.00 mm
- net Net-(J4-DAT2): track 0.00 -> 2.14 mm, vias 0 -> 1
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
Commit message: gah
Parts:
- removed D1, D2: PMEG2010ET, Package_TO_SOT_SMD:SOT-23
- removed R10: 111kR, Resistor_SMD:R_0402_1005Metric
- removed R9: 1MR, Resistor_SMD:R_0402_1005Metric
- added D5: PMEG2010ER, Diode_SMD:Nexperia_CFP3_SOD-123W, F.Cu at (121.8, 104.8)
- added D6: PMEG2010ER, Diode_SMD:Nexperia_CFP3_SOD-123W, F.Cu at (133.2, 93.0)
- C1, C2: value TBA -> 10pF
- C3, C4, C5, C6: footprint Capacitor_SMD:C_0201_0603Metric -> Capacitor_SMD:C_01005_0402Metric
- C30: footprint Capacitor_SMD:CP_Elec_8x10 -> Capacitor_THT:CP_Radial_D8.0mm_P3.50mm
- F1: footprint Fuse:Fuse_0402_1005Metric -> Fuse:Fuse_0603_1608Metric
- moved C30 1.58 mm to (129.2, 120.2)
- moved F1 0.28 mm to (140.4, 92.5)
Connections:
- C10 pad 1: Net-(U2-FB) -> V_OUT
- U2 pad 8: Net-(U2-FB) -> V_OUT
Routing:
- net Net-(D5-K): track 41.4 -> 11.2 mm
- net V_OUT: track 27.4 -> 39.0 mm, vias 2 -> 0
- net Net-(U2-FB): track 4.34 -> 0.00 mm
- net Net-(D6-A): track 9.55 -> 10.5 mm
- net GND: vias 81 -> 74
- net +16V8: vias 22 -> 23
Other:
- board text added: "AIAA, CSU Fresno Airbrakes Controller V1.0"
