File: rp2354b-fast.kicad_sch (KiCad schematic)
At the start: 22 parts, among them J2 Conn_ARM_SWD_TagConnect_TC203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, SW1 SW_Push, SW2 SW_Push, U1 RP2354B, Y1 12MHz

Commit message: routes
Parts:
- added C21, C22, C26, C27: 100nF, Capacitor_SMD:C_0402_1005Metric, symbol Device:C_Small
Connections:
- net +3V3: now also U1.15 (IOVDD), U1.24 (IOVDD), U1.29 (IOVDD), U1.41 (IOVDD), U1.5 (IOVDD), U1.50 (IOVDD), U1.59 (ADC_AVDD), U1.60 (IOVDD), U1.61 (VREG_AVDD), U1.68 (USB_OTP_VDD), U1.69 (QSPI_IOVDD), U1.76 (IOVDD), C21.1, C22.1, C26.1, C27.1
- net +DVDD: now also U1.10 (DVDD), U1.32 (DVDD), U1.51 (DVDD), U1.65 (VREG_FB)
- net GND: now also C21.2, C22.2, C26.2, C27.2; no longer U1.10 (DVDD), U1.15 (IOVDD), U1.24 (IOVDD), U1.29 (IOVDD), U1.32 (DVDD), U1.41 (IOVDD), U1.5 (IOVDD), U1.50 (IOVDD), U1.51 (DVDD), U1.59 (ADC_AVDD), U1.60 (IOVDD), U1.61 (VREG_AVDD), U1.65 (VREG_FB), U1.68 (USB_OTP_VDD), U1.69 (QSPI_IOVDD), U1.76 (IOVDD)
Other:
- sheet power_mng ports: added D+, D-; removed none
- moved on the sheet: C14, C15, C16, C17, C18, C19, C20, C23, C24, C25, SW1, SW2

Commit message: routes and bmp581
Parts:
- added C28, C29: 100nF, Capacitor_SMD:C_0402_1005Metric, symbol Device:C_Small
- added U4: BMP581, footprints:QFN10_BMP581_BOS-L, symbol BMP581:BMP581-10LGA
Connections:
- net +3V3: now also C29.2, U4.1 (VDDIO)
- net GND: now also C28.2, C29.1, U4.3 (V_SS), U4.8 (V_SS), U4.9 (V_SS)
- net GPIO16_SPI0_RX: now reaches U1.16 (GPIO16)
- net GPIO16_SPI0_RX: now also U4.5 (SDO)
- net GPIO17_SPI0_CSN: now reaches U1.17 (GPIO17)
- net GPIO17_SPI0_CSN: now also U4.6 (CSB)
- net GPIO18_SPI0_SCK: now reaches U1.18 (GPIO18)
- net GPIO18_SPI0_SCK: now also U4.2 (SCK)
- net GPIO19_SPI0_TX: now reaches U1.19 (GPIO19)
- net GPIO19_SPI0_TX: now also U4.4 (SDI)
- net GPIO20_SPI0_RX: now reaches U1.20 (GPIO20)
- net GPIO21_SPI0_CSN: now reaches U1.21 (GPIO21)
- net GPIO22SPI0_SCK: now reaches U1.22 (GPIO22)
- net GPIO23_SPI0_TX: now reaches U1.23 (GPIO23)
- new net: C28.1, U4.10 (V_DD)
- no-connect marks 8 -> 14
Other:
- moved on the sheet: D3

Commit message: hv16v
Parts:
- added U8: LSM9DS1, Package_LGA:LGA-24L_3x3.5mm_P0.43mm, symbol Sensor_Motion:LSM9DS1
- J2: value Conn_ARM_SWD_TagConnect_TC2030-NL -> TC2030-Tag
Connections:
- net ~{RESET}: no longer R3.2, SW2.2
- net GPIO33_LED: now reaches D3.3 (DIN)
- net GPIO33_LED: now also U1.42 (GPIO33)
- net STPER_ENABLE: now reaches U1.25 (GPIO24)
- net STPER_DIR: now reaches U1.26 (GPIO25)
- net STPER_STEP: now reaches U1.27 (GPIO26)
- net GPIO21_SPI0_CSN renamed GPIO21_SPIO_CSN
- net GPIO22SPI0_SCK renamed GPIO22_SPIO_SCK
- net GPIO23_SPI0_TX renamed GPIO23_SPIO_TX
- new net: R3.2, SW2.2
- new net: U8.1 (VDDIO), U8.3 (VDDIO)
- new net: U8.19 (GND), U8.20 (GND)
- new net: U8.22 (VDD), U8.23 (VDD)
Other:
- sheet power_mng renamed power_mng_3v3
- added sheet HV_16v8 (sch/HV_16v8.kicad_sch)
- moved on the sheet: C1, C14, C15, C16, C17, C18, C19, C2, C20, C21, C22, C23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

Commit message: imu sym
Parts:
- removed U8: LSM9DS1, Package_LGA:LGA-24L_3x3.5mm_P0.43mm, symbol Sensor_Motion:LSM9DS1
- added C39, C40: 100nF, Capacitor_SMD:C_0402_1005Metric, symbol Device:C_Small
- added U8: ISM6HG256X, Package_LGA:LGA-14_3x2.5mm_P0.5mm_LayoutBorder3x4y, symbol ISM6HG256X:ISM6HG256X
- U4: footprint footprints:QFN10_BMP581_BOS-L -> BMP581:QFN10_BMP581_BOS
Connections:
- net +3V3: now also C39.2, C40.2, U8.5 (VDDIO), U8.8 (VDD)
- net GND: now also C39.1, C40.1, U8.6 (GND), U8.7 (GND)
- net GPIO16_SPI0_RX: now also U8.1 (SDO/TA0)
- net GPIO18_SPI0_SCK: now also U8.13 (SCL)
- net GPIO19_SPI0_TX: now also U8.14 (SDA)
- net GPIO14_CSN_IMU: now reaches U1.14 (GPIO15)
- net GPIO14_CSN_IMU: now also U8.12 (CS)
- no-connect marks 14 -> 21
Other:
- sheet HV_16v8 ports: added DIR, ENABLE, SCLK, SDI, SDO, STEP, ~{SCS}; removed STPER_DIR, STPER_ENABLE, STPER_SCLK, STPER_SDI, STPER_SDO, STPER_STEP, STPER_~{SCS}
