File: rp2354b-fast.kicad_sch (KiCad schematic)
At the start: 32 parts, among them J2 TC2030-Tag, SW1 SW_Push, SW2 SW_Push, U1 RP2354B, U4 BMP581, U8 ISM6HG256X, Y1 12MHz

Commit message: MSD card, mag, imu
this thang gonna cost so much money
Parts:
- added C41: 1uF, Capacitor_SMD:C_0402_1005Metric, symbol Device:C_Small
- added C42, C44: 10uF, Capacitor_SMD:C_0402_1005Metric, symbol Device:C_Small
- added C43, C45: 100nF, Capacitor_SMD:C_0402_1005Metric, symbol Device:C_Small
- added H1, H2, H3, H4: MountingHole, MountingHole:MountingHole_3.2mm_M3, symbol Mechanical:MountingHole
- added J4: MSD-10-C, MSD-10-C:MSD-10-C, symbol MSD-10-C:MSD-10-C
- added R12, R13, R15, R16, R17, R18: 10kR, Resistor_SMD:R_0402_1005Metric, symbol Device:R_Small_US
- added U9: MMC5983MA, Package_LGA:LGA-16_3x3mm_P0.5mm, symbol MMC5983MA:MMC5983MA
Connections:
- net +3V3: now also C41.2, C43.2, C44.1, C45.1, J4.04 (VDD), R12.1, R13.1, R15.1, R16.1, R17.1, R18.1, U9.13 (VDDIO), U9.2 (VDD)
- net GND: now also C41.1, C42.1, C43.1, C44.2, C45.2, J4.06 (VSS), J4.G1 (COVER_GND), J4.G2 (COVER_GND__1), J4.G3 (COVER_GND__2), J4.G4 (COVER_GND__3), U9.11 (GND), U9.9 (GND)
- net GPIO16_SPI0_RX: now also J4.07 (DAT0), R15.2
- net GPIO18_SPI0_SCK: now also J4.05 (CLK), R16.2
- net GPIO19_SPI0_TX: now also J4.03 (CMD), R17.2
- net ~{RESET}: now also R3.2, SW2.2
- net GPIO28_SD_CS: now reaches U1.36 (GPIO28)
- net GPIO28_SD_CS: now also J4.02 (CD/DAT3), R18.2
- net GPIO36_RX: now reaches U1.45 (GPIO36)
- net GPIO36_RX: now also U9.5 (SPI_SDO)
- net GPIO37_CSN: now reaches U1.46 (GPIO37)
- net GPIO37_CSN: now also U9.4 (SPI_CS)
- net GPIO38_SCK: now reaches U1.47 (GPIO38)
- net GPIO38_SCK: now also U9.1 (SCL/SPI_SCK)
- net GPIO39_TX: now reaches U1.48 (GPIO39)
- net GPIO39_TX: now also U9.16 (SDA/SPI_SDI)
- new net: J4.01 (DAT2), R12.2
- new net: C42.2, U9.10 (CAP)
- new net: J4.08 (DAT1), R13.2
Other:
- moved on the sheet: D3

Commit message: gah
Parts:
- C1, C2: value TBA -> 10pF
Changed lines of the file:
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@@
 			)
 		)
-		(property "Value" "TBA"
+		(property "Value" "10pF"
 			(at 201.93 115.5762 0)
 			(show_name no)
@@
 			)
 		)
-		(property "Value" "TBA"
+		(property "Value" "10pF"
 			(at 175.26 115.5762 0)
 			(show_name no)

Commit message: reroute
doooom
Parts:
- added C47: 100nF, Capacitor_SMD:C_0402_1005Metric, symbol Device:C_Small
- added C48: 10uF, Capacitor_SMD:C_0402_1005Metric, symbol Device:C_Small
- added U11: SX1262, symbol WSCORE-SX1262:CORE1262
- SW1: value SW_Push -> BOOT
- SW2: value SW_Push -> RUN
Connections:
- net +3V3: now also C28.1, U1.64 (VREG_VIN), U4.10 (V_DD), C47.2, C48.2, U11.16 (3V3)
- net +DVDD: no longer U1.65 (VREG_FB)
- net GND: now also C1.2, C2.2, U1.65 (VREG_FB), C47.1, C48.1, U11.10 (GND), U11.15 (GND), U11.2 (GND), U11.9 (GND); no longer U1.64 (VREG_VIN)
- net GPIO16_SPI0_RX: now also U9.5 (SPI_SDO)
- net GPIO18_SPI0_SCK: now also U9.1 (SCL/SPI_SCK)
- net GPIO19_SPI0_TX: now also U9.16 (SDA/SPI_SDI)
- net GPIO28_CSN_BMP: now reaches U1.28 (GPIO27)
- net GPIO28_CSN_BMP: now also U4.6 (CSB)
- net GPIO14_CSN_IMU renamed GPIO14_CSN_SD
- net GPIO14_CSN_SD: now also J4.02 (CD/DAT3), R18.2; no longer U8.12 (CS)
- net GPIO17_SPI0_CSN renamed GPIO17_CSN_IMU
- net GPIO17_CSN_IMU: now also U8.12 (CS); no longer U4.6 (CSB)
- net GPIO21_SPIO_CSN renamed GPIO21_CSN_MAG
- net GPIO21_CSN_MAG: now also U9.4 (SPI_CS)
- removed net GPIO28_SD_CS: J4.02 (CD/DAT3), R18.2, U1.36 (GPIO28)
- net GPIO36_RX: no longer names the net of U1.45 (GPIO36)
- net GPIO36_RX: no longer U9.5 (SPI_SDO)
- net GPIO37_CSN: no longer names the net of U1.46 (GPIO37)
- net GPIO37_CSN: no longer U9.4 (SPI_CS)
- net GPIO38_SCK: no longer names the net of U1.47 (GPIO38)
- net GPIO38_SCK: no longer U9.1 (SCL/SPI_SCK)
- net GPIO39_TX: no longer names the net of U1.48 (GPIO39)
- net GPIO39_TX: no longer U9.16 (SDA/SPI_SDI)
- new net GPIO28_CSN_STPR: U1.36 (GPIO28)
- no-connect marks 21 -> 60
Other:
- note added: "GPIO36_RX"
- note added: "GPIO37_CSN"
- note added: "GPIO38_SCK"
- note added: "GPIO39_TX"
- moved on the sheet: C14, C15, C16, C17, C18, C19, C20, C21, C22, C23, C24, C25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

Commit message: v1.1c
sx1262 placement
need to route and assign pins
Parts:
- U11: footprint (none) -> WS-CORE-SX1262:CORE-1262
Changed lines of the file:
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@@
 			)
 		)
-		(property "Footprint" ""
+		(property "Footprint" "WS-CORE-SX1262:CORE-1262"
 			(at 109.22 163.83 0)
 			(hide yes)
