File: rp2354b-fast.kicad_sch (KiCad schematic)
At the start: 52 parts, among them J2 TC2030-Tag, J4 MSD-10-C, SW1 BOOT, SW2 RUN, U1 RP2354B, U11 SX1262, U4 BMP581, U8 ISM6HG256X, U9 MMC5983MA, Y1 12MHz

Commit message: sx1262 routes
routed!!
production ready??
Connections:
- net GPIO16_SPI0_RX: no longer J4.07 (DAT0), R15.2
- net GPIO18_SPI0_SCK: no longer J4.05 (CLK), R16.2
- net GPIO19_SPI0_TX: no longer J4.03 (CMD), R17.2
- net GPIO13_DIO1_RAD: now reaches U11.14 (DIO1)
- net GPIO13_DIO1_RAD: now also U1.12 (GPIO13)
- net GPIO12_CSN_RAD: now reaches U11.3 (CS)
- net GPIO12_CSN_RAD: now also U1.11 (GPIO12)
- net GPIO10_SPI1_SCK: now reaches U11.4 (CLK)
- net GPIO10_SPI1_SCK: now also J4.05 (CLK), R17.2, U1.8 (GPIO10)
- net GPIO11_SPI1_TX: now reaches U11.5 (MOSI)
- net GPIO11_SPI1_TX: now also J4.03 (CMD), R18.2, U1.9 (GPIO11)
- net GPIO08_SPI1_RX: now reaches U11.6 (MISO)
- net GPIO08_SPI1_RX: now also J4.07 (DAT0), R15.2, U1.6 (GPIO8)
- net GPIO15_RESET_RAD: now reaches U11.7 (RESET)
- net GPIO15_RESET_RAD: now also U1.14 (GPIO15)
- net GPIO14_BUSY_RAD: now reaches U11.8 (BUSY)
- net GPIO14_BUSY_RAD: now also U1.13 (GPIO14)
- net GPIO09_CSN_SD: now reaches U1.7 (GPIO9)
- net GPIO09_CSN_SD: now also J4.02 (CD/DAT3), R16.2
- removed net GPIO14_CSN_SD: J4.02 (CD/DAT3), R18.2, U1.14 (GPIO15)
- no-connect marks 60 -> 46
Other:
- note removed: "GPIO36_RX"
- note removed: "GPIO37_CSN"
- note removed: "GPIO38_SCK"
- note removed: "GPIO39_TX"
- moved on the sheet: C47, C48, U11

Commit message: v1.1d
ig bro
Parts:
- C1, C2: value 10pF -> TBA
Changed lines of the file:
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@@
 			)
 		)
-		(property "Value" "10pF"
+		(property "Value" "TBA"
 			(at 201.93 115.5762 0)
 			(show_name no)
@@
 			)
 		)
-		(property "Value" "10pF"
+		(property "Value" "TBA"
 			(at 175.26 115.5762 0)
 			(show_name no)

Commit message: footprints
Parts:
- added J7: Conn_01x06, Connector_PinHeader_2.54mm:PinHeader_1x06_P2.54mm_Vertical, symbol Connector_Generic:Conn_01x06
Connections:
- net at U1.43 (GPIO34): now also J7.1 (Pin_1)
- net at U1.44 (GPIO35): now also J7.2 (Pin_2)
- net at U1.45 (GPIO36): now also J7.3 (Pin_3)
- net at U1.46 (GPIO37): now also J7.4 (Pin_4)
- net at U1.47 (GPIO38): now also J7.5 (Pin_5)
- net at U1.48 (GPIO39): now also J7.6 (Pin_6)
- no-connect marks 46 -> 40
Changed lines of the file:
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@@
 	)
 	(no_connect
-		(at 260.35 144.78)
-	)
-	(no_connect
-		(at 260.35 139.7)
-	)
-	(no_connect
 		(at 260.35 50.8)
 	)
@@
 	)
 	(no_connect
-		(at 260.35 142.24)
-	)
-	(no_connect
 		(at 260.35 58.42)
 	)
@@
 	)
 	(no_connect
-		(at 260.35 137.16)
-	)
-	(no_connect
-		(at 260.35 149.86)
-	)
-	(no_connect
 		(at 209.55 149.86)
 	)
@@
 	)
 	(no_connect
-		(at 260.35 147.32)
-	)
-	(no_connect
 		(at 209.55 91.44)
 	)
@@
 	(wire
 		(pts
+			(xy 261.62 144.78) (xy 260.35 144.78)
+		)
+		(stroke
+			(width 0)
+			(type default)
+		)
+	)
+	(wire
+		(pts
 			(xy 242.57 43.18) (xy 242.57 35.56)
 		)
@@
 	(wire
 		(pts
+			(xy 261.62 149.86) (xy 260.35 149.86)
+		)
+		(stroke
+			(width 0)
+			(type default)
+		)
+	)
+	(wire
+		(pts
 			(xy 260.35 25.4) (xy 271.78 25.4)
 		)
@@
 	(wire
 		(pts
+			(xy 261.62 147.32) (xy 260.35 147.32)
+		)
+		(stroke
+			(width 0)
+			(type default)
+		)
+	)
+	(wire
+		(pts
 			(xy 100.33 106.68) (xy 130.81 106.68)
 		)
@@
 	(wire
 		(pts
+			(xy 261.62 137.16) (xy 260.35 137.16)
+		)
+		(stroke
+			(width 0)
+			(type default)
+		)
+	)
+	(wire
+		(pts
 			(xy 138.43 41.91) (xy 133.35 41.91)
 		)
@@
 	(wire
 		(pts
+			(xy 261.62 139.7) (xy 260.35 139.7)
+		)
+		(stroke
+			(width 0)
+			(type default)
+		)
+	)
+	(wire
+		(pts
 			(xy 25.4 77.47) (xy 40.64 77.47)
 		)
@@
 	(wire
 		(pts
+			(xy 261.62 142.24) (xy 260.35 142.24)
+		)
+		(stroke
+			(width 0)
+			(type default)
+		)
+	)
+	(wire
+		(pts
 			(xy 214.63 20.32) (xy 226.06 20.32)
 		)
@@
 					(unit 1)
 				)
+			)
+		)
+	)
+	(symbol
+		(lib_id "Connector_Generic:Conn_01x06")
+		(at 266.7 142.24 0)
+		(unit 1)
+		(body_style 1)
+		(exclude_from_sim no)
+		(in_bom yes)
+		(on_board yes)
+		(in_pos_files yes)
+		(dnp no)
+		(fields_autoplaced yes)
+		(property "Reference" "J7"
+			(at 269.24 142.2399 0)
+			(show_name no)
+			(do_not_autoplace no)
+			(effects
+				(font
+					(size 1.27 1.27)
+				)
+				(justify left)
+			)
+		)
+		(property "Value" "Conn_01x06"
+			(at 269.24 144.7799 0)
+			(show_name no)
+			(do_not_autoplace no)
+			(effects
+				(font
+					(size 1.27 1.27)
+				)
+				(justify left)
+			)
+		)
+		(property "Footprint" "Connector_PinHeader_2.54mm:PinHeader_1x06_P2.54mm_Vertical"
+			(at 266.7 142.24 0)
+			(hide yes)
+			(show_name no)
+			(do_not_autoplace no)
+			(effects
+				(font
+					(size 1.27 1.27)
+				)
+			)
+		)
+		(property "Datasheet" ""
+			(at 266.7 142.24 0)
+			(hide yes)
+			(show_name no)
+			(do_not_autoplace no)
+			(effects
+				(font
+					(size 1.27 1.27)
+				)
+			)
+		)
+		(property "Description" "Generic connector, single row, 01x06, script generated (kicad-library-utils/schlib/autogen/connector/)"
+			(at 266.7 142.24 0)
+			(hide yes)
+			(show_name no)
+			(do_not_autoplace no)
+			(effects
+				(font
+					(size 1.27 1.27)
+				)
+			)
+		)
+		(pin "3"
+		)
+		(pin "5"
+		)
+		(pin "6"
+		)
+		(pin "1"
+		)
+		(pin "4"
+		)
+		(pin "2"
+		)
+		(instances
+			(project "rp2354b-fast"
+				(path "/beb1ad91-9446-4312-87f0-5238465df71d"
+					(reference "J7")
+					(unit 1)
+				)

Commit message: v1.1e for real
ordered!
Redid high power side.
Added breakouts for power and the motor driver.
Parts:
- H1, H2, H3, H4: footprint MountingHole:MountingHole_3.2mm_M3 -> MountingHole:MountingHole_4.3mm_M4
- R12, R13, R15, R16, R17, R18: value 10kR -> 47kR
- R3: value 10kR -> 4.7kR
Changed lines of the file:
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@@
 			)
 		)
-		(property "Footprint" "MountingHole:MountingHole_3.2mm_M3"
+		(property "Footprint" "MountingHole:MountingHole_4.3mm_M4"
 			(at 193.04 43.18 0)
 			(hide yes)
@@
 			)
 		)
-		(property "Value" "10kR"
+		(property "Value" "47kR"
 			(at 114.3 69.8499 0)
 			(show_name no)
@@
 			)
 		)
-		(property "Value" "10kR"
+		(property "Value" "4.7kR"
 			(at 198.12 64.7699 0)
 			(show_name no)
@@
 			)
 		)
-		(property "Footprint" "MountingHole:MountingHole_3.2mm_M3"
+		(property "Footprint" "MountingHole:MountingHole_4.3mm_M4"
 			(at 193.04 48.26 0)
 			(hide yes)
@@
 			)
 		)
-		(property "Value" "10kR"
+		(property "Value" "47kR"
 			(at 107.95 102.8699 0)
 			(show_name no)
@@
 			)
 		)
-		(property "Value" "10kR"
+		(property "Value" "47kR"
 			(at 125.73 97.7899 0)
 			(show_name no)
@@
 			)
 		)
-		(property "Footprint" "MountingHole:MountingHole_3.2mm_M3"
+		(property "Footprint" "MountingHole:MountingHole_4.3mm_M4"
 			(at 175.26 43.18 0)
 			(hide yes)
@@
 			)
 		)
-		(property "Footprint" "MountingHole:MountingHole_3.2mm_M3"
+		(property "Footprint" "MountingHole:MountingHole_4.3mm_M4"
 			(at 175.26 48.26 0)
 			(hide yes)
@@
 			)
 		)
-		(property "Value" "10kR"
+		(property "Value" "47kR"
 			(at 119.38 64.7699 0)
 			(show_name no)
@@
 			)
 		)
-		(property "Value" "10kR"
+		(property "Value" "47kR"
 			(at 116.84 100.3299 0)
 			(show_name no)
@@
 			)
 		)
-		(property "Value" "10kR"
+		(property "Value" "47kR"
 			(at 97.79 105.4099 0)
 			(show_name no)
